File: Schematic/Nixie Clock/Nixie Circuit.sch (KiCad schematic (older format))
At the start: 0 parts

Commit message: Add files via upload
Parts:
- added C?: 10uF, Capacitor_SMD:C_0805_2012Metric_Pad1.15x1.40mm_HandSolder, symbol Device:CP
- added J6, J7, J8, J9: Conn_01x01_Female, Connector_PinHeader_2.00mm:PinHeader_1x01_P2.00mm_Vertical, symbol Connector:Conn_01x01_Female
- added J?: Conn_01x13_Female, Connector_PinHeader_2.00mm:PinHeader_1x13_P2.00mm_Vertical, symbol Connector:Conn_01x13_Female
- added M1, M2: 74141DIP16, Package_DIP:DIP-16_W7.62mm, symbol nixiemisc:74141DIP16
- added N1, N2, N3, N4: IN-16, Connector_PinHeader_2.00mm:PinHeader_2x06_P2.00mm_Vertical, symbol nixies-us:IN-16
- added R22, R25: 100R, Resistor_SMD:R_0201_0603Metric_Pad0.64x0.40mm_HandSolder, symbol Device:R
- added R23, R26: 470K, Resistor_SMD:R_0201_0603Metric_Pad0.64x0.40mm_HandSolder, symbol Device:R
- added R24, R27, R28, R29: 20K, Resistor_SMD:R_0201_0603Metric_Pad0.64x0.40mm_HandSolder, symbol Device:R
- added R?: 4K7, Resistor_SMD:R_0201_0603Metric_Pad0.64x0.40mm_HandSolder, symbol Device:R
- added TP?: 170V, TestPoint:TestPoint_Pad_1.5x1.5mm, symbol Connector:TestPoint
- added TP?: 5VD, TestPoint:TestPoint_Pad_1.5x1.5mm, symbol Connector:TestPoint
- added U8, U9: TLP627-1, Package_SO:SOP-4_3.8x4.1mm_P2.54mm, symbol Isolator:TLP521-1
- added U?: DC-DC 170V, Converter_DCDC:DCDC_2.5V_170V, symbol MCU_Module:DC-DC
- added U?: DC-DC 5V, Converter_DCDC:DCDC_2V~5V, symbol MCU_Module:DC-DC
Connections:
- new net: R22.1, U8.4
- new net: R25.1, U9.4
- new net: J6.1 (Pin_1), R24.2
- new net: J7.1 (Pin_1), R27.2
- new net: J8.1 (Pin_1), R28.2
- new net: J9.1 (Pin_1), R29.2
- new net: C?.1, R?.1, U?.1 (IN_PWR)
- new net 5VA: J?.9 (Pin_9), M1.5 (VCC), M2.5 (VCC), R?.2, U?.1 (IN_PWR)
- new net 5VD: J?.12 (Pin_12), TP?.1, U?.3 (OUT_PWR)
- new net DRIVER1A: J?.1 (Pin_1), M1.3 (A)
- new net DRIVER1B: J?.5 (Pin_5), M2.3 (A)
- new net DRIVER2A: J?.2 (Pin_2), M1.6 (B)
- new net DRIVER2B: J?.6 (Pin_6), M2.6 (B)
- new net DRIVER3A: J?.3 (Pin_3), M1.7 (C)
- new net DRIVER3B: J?.7 (Pin_7), M2.7 (C)
- new net DRIVER4A: J?.4 (Pin_4), M1.4 (D)
- new net DRIVER4B: J?.8 (Pin_8), M2.4 (D)
- new net GNDD: C?.2, J?.13 (Pin_13), M1.12 (GND), M2.12 (GND), R23.1, R26.1, U8.3, U9.3, U?.2 (IN_GND), U?.2 (IN_GND), U?.4 (OUT_GND), U?.4 (OUT_GND)
- new net GPIO4: J?.10 (Pin_10), R22.2
- new net GPIO5: J?.11 (Pin_11), R25.2
- new net HV: TP?.1, U8.1, U9.1, U?.3 (OUT_PWR)
- new net N1-3: N1.A, N3.A, R23.2, R24.1, R27.1, U8.2
- new net N1_0: M2.16 (0), N1.0, N3.0
- new net N1_1: M2.15 (1), N1.1, N3.1
- new net N1_2: M2.8 (2), N1.2, N3.2
- new net N1_3: M2.9 (3), N1.3, N3.3
- new net N1_4: M2.13 (4), N1.4, N3.4
- new net N1_5: M2.14 (5), N1.5, N3.5
- new net N1_6: M2.11 (6), N1.6, N3.6
- new net N1_7: M2.10 (7), N1.7, N3.7
- new net N1_8: M2.1 (8), N1.8, N3.8
- new net N1_9: M2.2 (9), N1.9, N3.9
- new net N2-4: N2.A, N4.A, R26.2, R28.1, R29.1, U9.2
- new net N2_0: M1.16 (0), N2.0, N4.0
- new net N2_1: M1.15 (1), N2.1, N4.1
- new net N2_2: M1.8 (2), N2.2, N4.2
- new net N2_3: M1.9 (3), N2.3, N4.3
- new net N2_4: M1.13 (4), N2.4, N4.4
- new net N2_5: M1.14 (5), N2.5, N4.5
- new net N2_6: M1.11 (6), N2.6, N4.6
- new net N2_7: M1.10 (7), N2.7, N4.7
- new net N2_8: M1.1 (8), N2.8, N4.8
- new net N2_9: M1.2 (9), N2.9, N4.9
