File: Schematic/Nixie Clock/Nixie Clock.sch (KiCad schematic (older format))
At the start: 53 parts

Commit message: Add files via upload
Parts:
- removed C?: C, symbol Device:C
- removed C?: CP, symbol Device:CP
- removed D?: BZD27Cxx, Diode_SMD:D_SMF, symbol Diode:BZD27Cxx
- removed FB?: Ferrite_Bead, symbol Device:Ferrite_Bead
- removed JP?: SolderJumper_2_Open, symbol Jumper:SolderJumper_2_Open
- removed P? (x3): DiscPiezo, symbol Piezo:DiscPiezo
- removed Q?: BC548, Package_TO_SOT_THT:TO-92_Inline, symbol Transistor_BJT:BC548
- removed Q?: BUZ11, Package_TO_SOT_THT:TO-220-3_Vertical, symbol Transistor_FET:BUZ11
- removed Q?: BC547, Package_TO_SOT_THT:TO-92_Inline, symbol Transistor_BJT:BC547
- removed RV?: R_POT, symbol Device:R_POT
- removed T?: Transformer_1P_1S, Transformer_SMD:Transformer_CEEH54_Nixie, symbol Device:Transformer_1P_1S
- removed U?: NE555D, Package_SO:SOIC-8_3.9x4.9mm_P1.27mm, symbol Timer:NE555D
- removed U?: DC-DC, symbol MCU_Module:DC-DC
- added C2, C4: 10uF, Capacitor_SMD:C_0805_2012Metric_Pad1.15x1.40mm_HandSolder, symbol Device:CP
- added C3: 20pF, Capacitor_SMD:C_0805_2012Metric_Pad1.15x1.40mm_HandSolder, symbol Device:C
- added D6, D7, D8: LED, Resistor_SMD:R_0805_2012Metric, symbol Device:LED
- added J1: Conn_02x02_Odd_Even, Connector_Molex:Molex_Nano-Fit_105310-xx04_2x02_P2.50mm_Vertical, symbol Connector_Generic:Conn_02x02_Odd_Even
- added J3, P2, P4: Conn_01x02_Female, Connector_PinHeader_2.00mm:PinHeader_1x02_P2.00mm_Vertical, symbol Connector:Conn_01x02_Female
- added J?: Conn_01x13_Female, Connector_PinHeader_2.00mm:PinHeader_1x13_P2.00mm_Vertical, symbol Connector:Conn_01x13_Female
- added R11: 1K2, Resistor_SMD:R_0201_0603Metric_Pad0.64x0.40mm_HandSolder, symbol Device:R
- added R12, R13, R16, R20: 1K, Resistor_SMD:R_0201_0603Metric_Pad0.64x0.40mm_HandSolder, symbol Device:R
- added R14: 100R, Resistor_SMD:R_0201_0603Metric_Pad0.64x0.40mm_HandSolder, symbol Device:R
- added U?: 74HC595, Package_DIP:DIP-16_W7.62mm, symbol 74xx:74HC595
- C1: renamed from C?; footprint (none) -> Capacitor_SMD:C_0805_2012Metric_Pad1.15x1.40mm_HandSolder
- C5: renamed from C?; value C -> 10uF; footprint (none) -> Capacitor_SMD:C_0805_2012Metric_Pad1.15x1.40mm_HandSolder
- C6: renamed from C?; value CP -> 10uF; footprint (none) -> Capacitor_SMD:C_0805_2012Metric_Pad1.15x1.40mm_HandSolder
- D1, D2: renamed from D?; footprint Diode_THT:D_DO-41_SOD81_P10.16mm_Horizontal -> Diode_SMD:D_SOD-523
- D5: renamed from D?; footprint (none) -> Package_TO_SOT_SMD:SOT-23
- FB1: renamed from FB?; footprint (none) -> Resistor_SMD:R_0201_0603Metric_Pad0.64x0.40mm_HandSolder
- J5: renamed from J?; footprint (none) -> Connector_PinHeader_2.00mm:PinHeader_2x03_P2.00mm_Vertical
- JP1: renamed from JP?; footprint (none) -> Jumper:SolderJumper-2_P1.3mm_Open_RoundedPad1.0x1.5mm
- P1: renamed from P?; footprint (none) -> Connector_USB:USB_C_Receptacle_XKB_U262-16XN-4BVC11
- Q1, Q2, Q4, Q5, Q6: renamed from Q?; footprint Package_TO_SOT_THT:TO-92_Inline -> Package_TO_SOT_SMD:SOT-23
- R1, R10, R15, R19, R2, R3, R4, R5, R6, R7, R8, R9: renamed from R?; footprint (none) -> Resistor_SMD:R_0201_0603Metric_Pad0.64x0.40mm_HandSolder
- R17: renamed from R?; value R -> 10K; footprint (none) -> Resistor_SMD:R_0201_0603Metric_Pad0.64x0.40mm_HandSolder
- R18: renamed from R?; footprint (none) -> Connector_PinHeader_2.00mm:PinHeader_1x02_P2.00mm_Vertical
- TP1: renamed from TP?; footprint (none) -> TestPoint:TestPoint_Pad_1.5x1.5mm
- U2: renamed from U?; footprint (none) -> Package_SO:MSOP-8-1EP_3x3mm_P0.65mm_EP1.95x2.15mm
- U3: renamed from U?; footprint (none) -> Package_TO_SOT_SMD:SOT-23-6
- U5: renamed from U?; footprint (none) -> Package_SO:TSSOP-8_3x3mm_P0.65mm
- gave numbers to parts that had none: 5
Connections:
- net DCDC is gone; now on net 5VA: Q2.3 (E)
- net 3.3VA: now also U?.10 (~SRCLR), U?.16 (VCC)
- net 5VA: now also U2.4 (VCC), U2.8 (CE), C2.1, D6.2 (A), D7.2 (A), D8.2 (A), J?.9 (Pin_9)
- net BAT1+: now also J1.2 (Pin_2), J3.1 (Pin_1), R14.2
- net GNDD: now also R17.2, U2.1 (TEMP), U2.3 (GND), C2.2, C4.1, J1.4 (Pin_4), J?.13 (Pin_13), P2.2 (Pin_2), P4.2 (Pin_2), R11.2, R16.1, U?.13 (~OE), U?.8 (GND)
- net MODE: now also P4.1 (Pin_1)
- net RX: now also J1.3 (Pin_3)
- net TX: now also J1.1 (Pin_1)
- net WAKE: now also P2.1 (Pin_1)
- net ANLDR: now reaches R17.1
- net ANLDR: now also R18.2, U1.17 (IO16)
- net at U2.2 (PROG): now also R11.1
- net BAT: now reaches U2.5 (BAT)
- net BAT: now also C4.2
- net at U2.6 (STDBY): now also R13.2
- net at U2.7 (CHRG): now also R12.2
- net G2: now reaches U3.1 (OD)
- net G2: now also U5.1 (S1)
- net G1: now reaches U3.3 (OC)
- net G1: now also U5.3 (S2)
- net at U3.4 (TD): now also R16.2
- net at U3.5 (VCC): now also C3.1, R14.1
- net at U3.6 (GND): now also C3.2
- net at U5.2 (D): now also U5.5 (D)
- net BAT1-: now reaches U5.6 (G1)
- net BAT1-: now also J3.2 (Pin_2)
- net PWLDR: now reaches R18.1
- net GPIO4: now reaches U1.10 (IO4)
- net GPIO4: now also J?.10 (Pin_10)
- net GPIO5: now reaches U1.14 (IO5)
- net GPIO5: now also J?.11 (Pin_11)
- net GPIO14: now reaches U1.3 (IO14)
- net GPIO14: now also U?.11 (SRCLK)
- net GPIO13: now reaches U1.5 (IO13)
- net GPIO13: now also U?.14 (SER)
- net GPIO15: now reaches U1.6 (IO15)
- net GPIO15: now also U?.12 (RCLK)
- new net: D8.1 (K), R20.1
- new net 5VD: J?.12 (Pin_12)
- new net CHRG: D6.1 (K), R12.1
- new net DRIVER1A: J?.1 (Pin_1), U?.15 (QA)
- new net DRIVER1B: J?.5 (Pin_5), U?.4 (QE)
- new net DRIVER2A: J?.2 (Pin_2), U?.1 (QB)
- new net DRIVER2B: J?.6 (Pin_6), U?.5 (QF)
- new net DRIVER3A: J?.3 (Pin_3), U?.2 (QC)
- new net DRIVER3B: J?.7 (Pin_7), U?.6 (QG)
- new net DRIVER4A: J?.4 (Pin_4), U?.3 (QD)
- new net DRIVER4B: J?.8 (Pin_8), U?.7 (QH)
- new net STDBY: D7.1 (K), R13.1
- new net WIFI: R20.2
Other:
- note added: "10K - 130mA\n5K - 250mA\n4K - 300mA\n3K - 400mA\n2K - 580mA\n1.66K - 690mA\n1.5K - 780mA\n1.33K - 900mA\n1.2K - 1A"
- moved on the sheet: C1, C5, C6, D1, D2, D3, D4, D5, FB1, J5, JP1, P1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
