File: Projeto Relogio Nixie IN17.kicad_sch (KiCad schematic)
At the start: 73 parts, among them J1 nixie0, J2 nixie1, J3 BATTERY, J4 UART, P1 USB_C_Plug, Q1 BC817, Q2 STD17NF25, Q3 BC817, Q4 BC548, Q5 2N7000, Q6 BC548, Q7 BC548, Q8 BC548, SW1 SW_Push, SW2 SW_Push, SW3 SPST_B3U-1000P, SW4 SPST_B3U-1000P, U1 MAX1771xSA, U2 CP2102N-A01-GQFN24, U3 HV5523K7-G, U4 PAM2305AABADJ, U5 MCP73831-3-OT, U6 ESP32-PICO-D4

Commit message: Add files via upload
Parts:
- removed AE1: Antenna, ESP_Antenna:ESPRESSIF_ESP32_MIFA_2.4GHz_Right, symbol Device:Antenna
- removed C8: 47uF, Capacitor_SMD:C_0805_2012Metric, symbol Device:C
- removed D3: DZ2S056X0L, Diode_SMD:D_2114_3652Metric, symbol Diode:DZ2S056X0L
- removed J1: nixie0, Connector_PinHeader_1.27mm:PinHeader_2x06_P1.27mm_Vertical, symbol Connector_Generic:Conn_01x12
- removed J2: nixie1, Connector_PinHeader_1.27mm:PinHeader_2x06_P1.27mm_Vertical, symbol Connector_Generic:Conn_01x12
- removed J4: UART, Connector_PinHeader_2.00mm:PinHeader_1x03_P2.00mm_Vertical, symbol Projeto Relogio Pulso 2Displays-rescue:Conn_01x03_Male-Connector
- removed JP1: ~, Jumper:SolderJumper-2_P1.3mm_Open_RoundedPad1.0x1.5mm, symbol Jumper:SolderJumper_2_Open
- removed P1: USB_C_Plug, Connector_USB:USB_C_Receptacle_Palconn_UTC16-G, symbol Connector:USB_C_Plug
- removed Q5: 2N7000, Package_TO_SOT_SMD:SOT-23, symbol Transistor_FET:2N7000
- removed Q6: BC548, Package_TO_SOT_SMD:SOT-23, symbol Transistor_BJT:BC548
- removed R14: 2K2, Resistor_SMD:R_0603_1608Metric, symbol Device:R
- removed R15, R19: 4K7, Resistor_SMD:R_0603_1608Metric, symbol Device:R
- removed R21: 1M, Resistor_SMD:R_0603_1608Metric, symbol Device:R
- removed R7: 15K, Resistor_SMD:R_0603_1608Metric, symbol Device:R
- removed TP1: 5VA, TestPoint:TestPoint_Pad_1.5x1.5mm, symbol Connector:TestPoint
- added J1: Conn_01x04, Connector:Magnetic_01x04, symbol Connector_Generic:Conn_01x04
- added J2, J3: Conn_01x24, Connector_PinHeader_1.27mm:PinHeader_2x12_P1.27mm_Vertical, symbol Connector_Generic:Conn_01x24
- added J5: ANTENNA, Connector_PinHeader_2.00mm:PinHeader_1x02_P2.00mm_Vertical, symbol Connector_Generic:Conn_01x02
- added N1, N2: IN-16, nixies-us:nixies-us-IN-16, symbol nixies-us:IN-16
- added R5: 15K, Resistor_SMD:R_0603_1608Metric, symbol Device:R
- renumbered C11 to C10, C12 to C11, C13 to C12, C9 to C8, C10 to C9, D4 to D3, D5 to D4, D6 to D5, D7 to D6, J3 to J4, Q7 to Q5, Q8 to Q6, R16 to R14, R17 to R15, R18 to R16, R20 to R17, R22 to R18, R23 to R19, R24 to R20, R25 to R21, R5 to R6, R6 to R7
Connections:
- net ANT: now also J5.2 (Pin_2)
- net GNDD: now also J1.4 (Pin_4), J5.1 (Pin_1)
- net HV: now also J2.1 (Pin_1), J2.2 (Pin_2); no longer R11.1
- net IN0_0: now also J3.14 (Pin_14), N1.0; no longer U3.1 (HVOUT11)
- net IN0_1: now also J3.18 (Pin_18), N1.1; no longer U3.2 (HVOUT12)
- net IN0_2: now also J3.8 (Pin_8), N1.2; no longer U3.3 (HVOUT13)
- net IN0_3: now also J3.20 (Pin_20), N1.3; no longer U3.4 (HVOUT14)
- net IN0_4: now also J3.16 (Pin_16), N1.4; no longer U3.5 (HVOUT15)
- net IN0_5: now also J3.12 (Pin_12), N1.5; no longer U3.6 (HVOUT16)
- net IN0_6: now also J3.10 (Pin_10), N1.6; no longer U3.7 (HVOUT17)
- net IN0_7: now also J3.22 (Pin_22), N1.7; no longer U3.8 (HVOUT18)
- net IN0_8: now also J3.4 (Pin_4), N1.8; no longer U3.9 (HVOUT19)
- net IN0_9: now also J3.6 (Pin_6), N1.9; no longer U3.10 (HVOUT20)
- net IN1_0: now also J3.13 (Pin_13), N2.0; no longer U3.12 (HVOUT22)
- net IN1_1: now also J3.17 (Pin_17), N2.1; no longer U3.13 (HVOUT23)
- net IN1_2: now also J3.7 (Pin_7), N2.2; no longer U3.14 (HVOUT24)
- net IN1_3: now also J3.19 (Pin_19), N2.3; no longer U3.15 (HVOUT25)
- net IN1_4: now also J3.15 (Pin_15), N2.4; no longer U3.16 (HVOUT26)
- net IN1_5: now also J3.11 (Pin_11), N2.5; no longer U3.17 (HVOUT27)
- net IN1_6: now also J3.9 (Pin_9), N2.6; no longer U3.18 (HVOUT28)
- net IN1_7: now also J3.21 (Pin_21), N2.7; no longer U3.19 (HVOUT29)
- net IN1_8: now also J3.3 (Pin_3), N2.8; no longer U3.20 (HVOUT30)
- net IN1_9: now also J3.5 (Pin_5), N2.9; no longer U3.21 (HVOUT31)
- net RX0: now also J1.2 (Pin_2)
- net TX0: now also J1.3 (Pin_3)
- net VIN: now also J1.1 (Pin_1)
- net at R11.2: now also N2.A
- net IN0_DP: no longer names the net of U3.11 (HVOUT21)
- net IN0_DP: now also J2.14 (Pin_14)
- net IN1_DP: no longer names the net of U3.22 (HVOUT32)
- net IN1_DP: now also J2.3 (Pin_3)
- new net: N1.A, R5.2
- new net: J2.24 (Pin_24), U3.1 (HVOUT11)
- new net: J2.15 (Pin_15), U3.10 (HVOUT20)
- new net: J2.13 (Pin_13), U3.12 (HVOUT22)
- new net: J2.12 (Pin_12), U3.13 (HVOUT23)
- new net: J2.11 (Pin_11), U3.14 (HVOUT24)
- new net: J2.10 (Pin_10), U3.15 (HVOUT25)
- new net: J2.9 (Pin_9), U3.16 (HVOUT26)
- new net: J2.8 (Pin_8), U3.17 (HVOUT27)
- new net: J2.7 (Pin_7), U3.18 (HVOUT28)
- new net: J2.6 (Pin_6), U3.19 (HVOUT29)
- new net: J2.23 (Pin_23), U3.2 (HVOUT12)
- new net: J2.5 (Pin_5), U3.20 (HVOUT30)
- new net: J2.4 (Pin_4), U3.21 (HVOUT31)
- new net: J2.22 (Pin_22), U3.3 (HVOUT13)
- new net: J2.21 (Pin_21), U3.4 (HVOUT14)
- new net: J2.20 (Pin_20), U3.5 (HVOUT15)
- new net: J2.19 (Pin_19), U3.6 (HVOUT16)
- new net: J2.18 (Pin_18), U3.7 (HVOUT17)
- new net: J2.17 (Pin_17), U3.8 (HVOUT18)
- new net: J2.16 (Pin_16), U3.9 (HVOUT19)
- new net HVe: J3.23 (Pin_23), J3.24 (Pin_24), R11.1, R5.1
- new net IN0_LHDP: J3.2 (Pin_2)
- new net IN0_LHDPe: N1.LHDP
- new net IN1_RHDP: J3.1 (Pin_1)
- new net IN1_RHDPe: N2.RHDP
Other:
- note removed: "Circuito de Entrada com Proteção de Sobretensão 5.6Vmax"

Commit message: Add files via upload
Parts:
- removed J2: Conn_01x24, Connector_PinHeader_1.27mm:PinHeader_2x12_P1.27mm_Vertical, symbol Connector_Generic:Conn_01x24
- added J2: Conn_02x12_Odd_Even, Connector_PinHeader_1.27mm:PinHeader_2x12_P1.27mm_Vertical, symbol Connector_Generic:Conn_02x12_Odd_Even
- J3: symbol Connector_Generic:Conn_01x24 -> Connector_Generic:Conn_02x12_Odd_Even
Connections:
- net HV: now also J2.1 (Pin_1), J2.2 (Pin_2)
- net IN0_0: now also J3.15 (Pin_15); no longer J3.14 (Pin_14)
- net IN0_1: now also J3.17 (Pin_17); no longer J3.18 (Pin_18)
- net IN0_2: now also J3.14 (Pin_14); no longer J3.8 (Pin_8)
- net IN0_3: now also J3.21 (Pin_21); no longer J3.20 (Pin_20)
- net IN0_4: now also J3.20 (Pin_20); no longer J3.16 (Pin_16)
- net IN0_5: now also J3.18 (Pin_18); no longer J3.12 (Pin_12)
- net IN0_6: now also J3.16 (Pin_16); no longer J3.10 (Pin_10)
- net IN0_7: now also J3.19 (Pin_19); no longer J3.22 (Pin_22)
- net IN0_8: now also J3.11 (Pin_11); no longer J3.4 (Pin_4)
- net IN0_9: now also J3.13 (Pin_13); no longer J3.6 (Pin_6)
- net IN0_LHDP: now also J3.1 (Pin_1); no longer J3.2 (Pin_2)
- net IN1_0: now also J3.6 (Pin_6); no longer J3.13 (Pin_13)
- net IN1_1: now also J3.8 (Pin_8); no longer J3.17 (Pin_17)
- net IN1_2: now also J3.3 (Pin_3); no longer J3.7 (Pin_7)
- net IN1_3: now also J3.12 (Pin_12); no longer J3.19 (Pin_19)
- net IN1_4: now also J3.9 (Pin_9); no longer J3.15 (Pin_15)
- net IN1_5: now also J3.7 (Pin_7); no longer J3.11 (Pin_11)
- net IN1_6: now also J3.5 (Pin_5); no longer J3.9 (Pin_9)
- net IN1_7: now also J3.10 (Pin_10); no longer J3.21 (Pin_21)
- net IN1_8: now also J3.2 (Pin_2); no longer J3.3 (Pin_3)
- net IN1_9: now also J3.4 (Pin_4); no longer J3.5 (Pin_5)
- net IN1_RHDP: now also J3.22 (Pin_22); no longer J3.1 (Pin_1)
- net HVOUT11: now reaches U3.1 (HVOUT11)
- net HVOUT11: now also J2.23 (Pin_23)
- net HVOUT20: now reaches U3.10 (HVOUT20)
- net HVOUT20: now also J2.5 (Pin_5)
- net HVOUT21: now reaches U3.11 (HVOUT21)
- net HVOUT21: now also J2.3 (Pin_3)
- net HVOUT22: now reaches U3.12 (HVOUT22)
- net HVOUT22: now also J2.4 (Pin_4)
- net HVOUT23: now reaches U3.13 (HVOUT23)
- net HVOUT23: now also J2.6 (Pin_6)
- net HVOUT24: now reaches U3.14 (HVOUT24)
- net HVOUT24: now also J2.8 (Pin_8)
- net HVOUT25: now reaches U3.15 (HVOUT25)
- net HVOUT25: now also J2.10 (Pin_10)
- net HVOUT26: now reaches U3.16 (HVOUT26)
- net HVOUT26: now also J2.12 (Pin_12)
- net HVOUT27: now reaches U3.17 (HVOUT27)
- net HVOUT27: now also J2.14 (Pin_14)
- net HVOUT28: now reaches U3.18 (HVOUT28)
- net HVOUT28: now also J2.16 (Pin_16)
- net HVOUT29: now reaches U3.19 (HVOUT29)
- net HVOUT29: now also J2.18 (Pin_18)
- net HVOUT12: now reaches U3.2 (HVOUT12)
- net HVOUT12: now also J2.21 (Pin_21)
- net HVOUT30: now reaches U3.20 (HVOUT30)
- net HVOUT30: now also J2.20 (Pin_20)
- net HVOUT31: now reaches U3.21 (HVOUT31)
- net HVOUT31: now also J2.22 (Pin_22)
- net HVOUT32: now reaches U3.22 (HVOUT32)
- net HVOUT32: now also J2.24 (Pin_24)
- net HVOUT13: now reaches U3.3 (HVOUT13)
- net HVOUT13: now also J2.19 (Pin_19)
- net HVOUT14: now reaches U3.4 (HVOUT14)
- net HVOUT14: now also J2.17 (Pin_17)
- net HVOUT15: now reaches U3.5 (HVOUT15)
- net HVOUT15: now also J2.15 (Pin_15)
- net HVOUT16: now reaches U3.6 (HVOUT16)
- net HVOUT16: now also J2.13 (Pin_13)
- net HVOUT17: now reaches U3.7 (HVOUT17)
- net HVOUT17: now also J2.11 (Pin_11)
- net HVOUT18: now reaches U3.8 (HVOUT18)
- net HVOUT18: now also J2.9 (Pin_9)
- net HVOUT19: now reaches U3.9 (HVOUT19)
- net HVOUT19: now also J2.7 (Pin_7)
Other:
- moved on the sheet: J3

Commit message: Add files via upload
Parts:
- removed J3: Conn_01x24, Connector_PinHeader_1.27mm:PinHeader_2x12_P1.27mm_Vertical, symbol Connector_Generic:Conn_02x12_Odd_Even
- added J3: Conn_01x24, Connector_FFC-FPC:TE_2-1734839-4_1x24-1MP_P0.5mm_Horizontal, symbol Connector_Generic:Conn_01x24
- J2: footprint Connector_PinHeader_1.27mm:PinHeader_2x12_P1.27mm_Vertical -> Connector_FFC-FPC:TE_2-1734839-4_1x24-1MP_P0.5mm_Horizontal; symbol Connector_Generic:Conn_02x12_Odd_Even -> Connector_Generic:Conn_01x24
Connections:
- net HV: now also J2.24 (Pin_24); no longer J2.2 (Pin_2)
- net HVOUT11: now also J2.2 (Pin_2); no longer J2.23 (Pin_23)
- net HVOUT12: now also J2.3 (Pin_3); no longer J2.21 (Pin_21)
- net HVOUT13: now also J2.4 (Pin_4); no longer J2.19 (Pin_19)
- net HVOUT14: now also J2.5 (Pin_5); no longer J2.17 (Pin_17)
- net HVOUT15: now also J2.6 (Pin_6); no longer J2.15 (Pin_15)
- net HVOUT16: now also J2.7 (Pin_7); no longer J2.13 (Pin_13)
- net HVOUT17: now also J2.8 (Pin_8); no longer J2.11 (Pin_11)
- net HVOUT19: now also J2.10 (Pin_10); no longer J2.7 (Pin_7)
- net HVOUT20: now also J2.11 (Pin_11); no longer J2.5 (Pin_5)
- net HVOUT21: now also J2.12 (Pin_12); no longer J2.3 (Pin_3)
- net HVOUT22: now also J2.13 (Pin_13); no longer J2.4 (Pin_4)
- net HVOUT23: now also J2.14 (Pin_14); no longer J2.6 (Pin_6)
- net HVOUT24: now also J2.15 (Pin_15); no longer J2.8 (Pin_8)
- net HVOUT25: now also J2.16 (Pin_16); no longer J2.10 (Pin_10)
- net HVOUT26: now also J2.17 (Pin_17); no longer J2.12 (Pin_12)
- net HVOUT27: now also J2.18 (Pin_18); no longer J2.14 (Pin_14)
- net HVOUT28: now also J2.19 (Pin_19); no longer J2.16 (Pin_16)
- net HVOUT29: now also J2.20 (Pin_20); no longer J2.18 (Pin_18)
- net HVOUT30: now also J2.21 (Pin_21); no longer J2.20 (Pin_20)
- net HVOUT32: now also J2.23 (Pin_23); no longer J2.24 (Pin_24)
- net HVe: now also J3.1 (Pin_1), J3.24 (Pin_24)
- net IN0_0: now also J3.23 (Pin_23)
- net IN0_1: now also J3.22 (Pin_22)
- net IN0_2: now also J3.14 (Pin_14)
- net IN0_3: now also J3.20 (Pin_20)
- net IN0_4: now also J3.17 (Pin_17)
- net IN0_5: now also J3.16 (Pin_16)
- net IN0_6: now also J3.15 (Pin_15)
- net IN0_7: now also J3.21 (Pin_21)
- net IN0_8: now also J3.18 (Pin_18)
- net IN0_9: now also J3.19 (Pin_19)
- net IN0_LHDPe: now also J3.13 (Pin_13)
- net IN1_0: now also J3.9 (Pin_9)
- net IN1_1: now also J3.8 (Pin_8)
- net IN1_2: now also J3.2 (Pin_2)
- net IN1_3: now also J3.6 (Pin_6)
- net IN1_4: now also J3.5 (Pin_5)
- net IN1_5: now also J3.4 (Pin_4)
- net IN1_6: now also J3.3 (Pin_3)
- net IN1_7: now also J3.7 (Pin_7)
- net IN1_8: now also J3.11 (Pin_11)
- net IN1_9: now also J3.10 (Pin_10)
- net IN1_RHDPe: now also J3.12 (Pin_12)
Other:
- moved on the sheet: J2

Commit message: Add files via upload
Parts:
- added C2: 100uF, Capacitor_Tantalum_SMD:CP_EIA-1608-08_AVX-J, symbol Device:C_Polarized
- added D2, D3: 1N4148W, Diode_SMD:D_SOD-123, symbol Diode:1N4148W
- renumbered C9 to C10, C10 to C11, C11 to C12, C12 to C13, C2 to C3, C3 to C4, C4 to C5, C5 to C6, C6 to C7, C7 to C8, C8 to C9, D2 to D4, D3 to D5, D4 to D6, D5 to D7, D6 to D8, J3 to J2, J2 to J3
Connections:
- net IO0 is gone; now on net BOOT: Q3.2 (E)
- net GNDD: now also C2.2
- net VIN: now also C2.1, D2.1 (K), D3.1 (K); no longer J1.1 (Pin_1)
- new net: D2.2 (A), D3.2 (A), J1.1 (Pin_1)
Other:
- moved on the sheet: J1
