File: Projeto Relogio Nixie IN17.kicad_pcb (KiCad board)
At the start: 2 copper layers, 50 x 50 mm, 73 parts, among them J1 nixie0, J2 nixie1, J3 BATTERY, J4 UART, P1 USB_C_Plug, Q1 BC817, Q2 STD17NF25, Q3 BC817, Q4 BC548, Q5 2N7000, Q6 BC548, Q7 BC548, Q8 BC548, SW1 SW_Push, SW2 SW_Push, SW3 SPST_B3U-1000P, SW4 SPST_B3U-1000P, U1 MAX1771xSA, U2 CP2102N-A01-GQFN24, U3 HV5523K7-G, U4 PAM2305AABADJ, U5 MCP73831-3-OT, U6 ESP32-PICO-D4

Commit message: Add files via upload
Parts:
- removed AE1: Antenna, ESP_Antenna:ESPRESSIF_ESP32_MIFA_2.4GHz_Right
- removed the C8 at (131.2, 58.4)
- removed the D4 at (125.5, 67.7)
- removed the J4 at (78.9, 45.4)
- removed P1: USB_C_Plug, Connector_USB:USB_C_Receptacle_Palconn_UTC16-G
- removed Q7, Q8: BC548, Package_TO_SOT_SMD:SOT-23
- removed the R15 at (115.8, 62.7)
- removed the R18 at (131.5, 71.9)
- removed the R19 at (118.0, 58.4)
- removed the R20 at (130.5, 67.7)
- removed the R21 at (120.4, 58.4)
- removed the R7 at (59.5, 78.0)
- added J3: Conn_01x24, Connector_PinHeader_1.27mm:PinHeader_2x12_P1.27mm_Vertical, F.Cu at (150.4, 90.2)
- added J5: ANTENNA, Connector_PinHeader_2.00mm:PinHeader_1x02_P2.00mm_Vertical, F.Cu at (126.6, 45.4)
- added N1: IN-16, nixies-us:nixies-us-IN-16, F.Cu at (135.9, 99.6)
- added N2: IN-16, nixies-us:nixies-us-IN-16, F.Cu at (149.3, 99.6)
- added R17: 100R, Resistor_SMD:R_0603_1608Metric, B.Cu at (147.8, 61.5)
- added R5: 15K, Resistor_SMD:R_0603_1608Metric, B.Cu at (135.9, 99.6)
- C1, R11, U2: moved to B.Cu
- C10: renamed from C11; moved to B.Cu
- C11: renamed from C12; moved to B.Cu
- D3: value DZ2S056X0L -> BZD27Cxx; moved to F.Cu
- J1: value nixie0 -> Conn_01x04; footprint Connector_PinHeader_1.27mm:PinHeader_2x06_P1.27mm_Vertical -> Connector:Magnetic_01x04
- J2: value nixie1 -> Conn_01x24; footprint Connector_PinHeader_1.27mm:PinHeader_2x06_P1.27mm_Vertical -> Connector_PinHeader_1.27mm:PinHeader_2x12_P1.27mm_Vertical
- JP1, Q4, R13, U5: moved to F.Cu
- Q5: value 2N7000 -> BC548
- R14: value 2K2 -> 1K
- R15: renamed from R17; moved to F.Cu
- moved R19 93.9 mm to (130.0, 79.9), turned to 45 degrees
- moved D4 93.9 mm to (130.0, 80.0), turned to 45 degrees
- moved SW3 92.7 mm to (135.5, 41.0), turned to -65 degrees
- moved R18 92.6 mm to (135.4, 41.0), turned to -65 degrees
- moved D5 90.9 mm to (128.0, 78.0), turned to 45 degrees
- moved R20 90.9 mm to (128.0, 78.0), turned to -135 degrees
- moved SW4 90.0 mm to (132.3, 42.5), turned to -65 degrees
- moved C12 89.9 mm to (132.2, 42.5), turned to -65 degrees
- moved D6 88.2 mm to (126.0, 76.0), turned to 45 degrees
- moved R21 88.2 mm to (126.0, 76.0), turned to -135 degrees
- moved U6 87.2 mm to (141.5, 57.5), turned to 45 degrees
- moved R9 84.1 mm to (125.9, 51.0)
- moved SW2 84.1 mm to (124.0, 48.8)
- moved SW1 84.0 mm to (121.7, 53.7), turned to -15 degrees
- moved R8 83.0 mm to (124.0, 55.3), turned to 75 degrees
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- renumbered C13 to C12, C9 to C8, C10 to C9, D5 to D4, D6 to D5, D7 to D6, J3 to J4, R22 to R18, R23 to R19, R24 to R20, R25 to R21, R5 to R6, R6 to R7
Connections:
- net IN1_6 renamed Net-(J2-Pin_7)
- D3 pad 2: BAT- -> Net-(D3-A)
- J1 pad 1: IN0_0 -> VIN
- J1 pad 2: IN0_1 -> RX0
- J1 pad 3: IN0_2 -> TX0
- J1 pad 4: IN0_3 -> BAT-
- J2 pad 1: IN1_0 -> HV
- J2 pad 10: IN1_9 -> Net-(J2-Pin_10)
- J2 pad 11: IN1_DP -> Net-(J2-Pin_11)
- J2 pad 2: IN1_1 -> HV
- J2 pad 3: IN1_2 -> Net-(J2-Pin_3)
- J2 pad 4: IN1_3 -> Net-(J2-Pin_4)
- J2 pad 5: IN1_4 -> Net-(J2-Pin_5)
- J2 pad 6: IN1_5 -> Net-(J2-Pin_6)
- J2 pad 8: IN1_7 -> Net-(J2-Pin_8)
- J2 pad 9: IN1_8 -> Net-(J2-Pin_9)
- Q5 pad 1: 5VA -> Net-(Q4-B)
- Q5 pad 2: Net-(Q5-G) -> Net-(Q5-B)
- Q5 pad 3: VIN -> BAT-
- Q6 pad 1: VIN -> Net-(Q6-C)
- Q6 pad 3: Net-(Q5-G) -> BAT-
- R11 pad 1: HV -> HVe
- R11 pad 2: Net-(J2-Pin_12) -> Net-(N2-PadA)
- R12 pad 2: Net-(Q8-C) -> Net-(Q6-C)
- R14 pad 1: VIN -> Net-(Q5-B)
- R14 pad 2: Net-(R14-Pad2) -> Net-(Q6-C)
- R16 pad 1: Net-(Q7-B) -> Net-(Q6-B)
- R16 pad 2: Net-(Q8-C) -> Net-(D3-A)
- U3 pad 1: IN0_0 -> Net-(J2-Pin_24)
- U3 pad 10: IN0_9 -> Net-(J2-Pin_15)
- U3 pad 11: IN0_DP -> Net-(J2-Pin_14)
- U3 pad 12: IN1_0 -> Net-(J2-Pin_13)
- U3 pad 13: IN1_1 -> Net-(J2-Pin_12)
- U3 pad 14: IN1_2 -> Net-(J2-Pin_11)
- U3 pad 15: IN1_3 -> Net-(J2-Pin_10)
- U3 pad 16: IN1_4 -> Net-(J2-Pin_9)
- U3 pad 17: IN1_5 -> Net-(J2-Pin_8)
- U3 pad 19: IN1_7 -> Net-(J2-Pin_6)
- U3 pad 2: IN0_1 -> Net-(J2-Pin_23)
- U3 pad 20: IN1_8 -> Net-(J2-Pin_5)
- U3 pad 21: IN1_9 -> Net-(J2-Pin_4)
- U3 pad 22: IN1_DP -> Net-(J2-Pin_3)
- U3 pad 3: IN0_2 -> Net-(J2-Pin_22)
- U3 pad 4: IN0_3 -> Net-(J2-Pin_21)
- U3 pad 5: IN0_4 -> Net-(J2-Pin_20)
- U3 pad 6: IN0_5 -> Net-(J2-Pin_19)
- U3 pad 7: IN0_6 -> Net-(J2-Pin_18)
- U3 pad 8: IN0_7 -> Net-(J2-Pin_17)
- U3 pad 9: IN0_8 -> Net-(J2-Pin_16)
Routing:
- added copper zone on B.Cu, net BAT-
- added copper zone on F.Cu, net BAT-
Other:
- board size 50 x 50 mm -> 49.8 x 67.6 mm

Commit message: Add files via upload
Parts:
- J2: value Conn_01x24 -> Conn_02x12_Odd_Even
- moved J3 0.78 mm to (150.2, 91.0)
- moved J2 0.61 mm to (136.0, 80.3)
Connections:
- net Net-(J2-Pin_10) renamed HVOUT25
- J2 pad 11: Net-(J2-Pin_11) -> HVOUT17
- J2 pad 12: Net-(J2-Pin_12) -> HVOUT26
- J2 pad 13: Net-(J2-Pin_13) -> HVOUT16
- J2 pad 14: Net-(J2-Pin_14) -> HVOUT27
- J2 pad 15: Net-(J2-Pin_15) -> HVOUT15
- J2 pad 16: Net-(J2-Pin_16) -> HVOUT28
- J2 pad 17: Net-(J2-Pin_17) -> HVOUT14
- J2 pad 18: Net-(J2-Pin_18) -> HVOUT29
- J2 pad 19: Net-(J2-Pin_19) -> HVOUT13
- J2 pad 20: Net-(J2-Pin_20) -> HVOUT30
- J2 pad 21: Net-(J2-Pin_21) -> HVOUT12
- J2 pad 22: Net-(J2-Pin_22) -> HVOUT31
- J2 pad 23: Net-(J2-Pin_23) -> HVOUT11
- J2 pad 24: Net-(J2-Pin_24) -> HVOUT32
- J2 pad 3: Net-(J2-Pin_3) -> HVOUT21
- J2 pad 4: Net-(J2-Pin_4) -> HVOUT22
- J2 pad 5: Net-(J2-Pin_5) -> HVOUT20
- J2 pad 6: Net-(J2-Pin_6) -> HVOUT23
- J2 pad 7: Net-(J2-Pin_7) -> HVOUT19
- J2 pad 8: Net-(J2-Pin_8) -> HVOUT24
- J2 pad 9: Net-(J2-Pin_9) -> HVOUT18
- J3 pad 1: IN1_RHDP -> IN0_LHDP
- J3 pad 10: IN0_6 -> IN1_7
- J3 pad 11: IN1_5 -> IN0_8
- J3 pad 12: IN0_5 -> IN1_3
- J3 pad 13: IN1_0 -> IN0_9
- J3 pad 14: IN0_0 -> IN0_2
- J3 pad 15: IN1_4 -> IN0_0
- J3 pad 16: IN0_4 -> IN0_6
- J3 pad 17: IN1_1 -> IN0_1
- J3 pad 18: IN0_1 -> IN0_5
- J3 pad 19: IN1_3 -> IN0_7
- J3 pad 2: IN0_LHDP -> IN1_8
- J3 pad 20: IN0_3 -> IN0_4
- J3 pad 21: IN1_7 -> IN0_3
- J3 pad 22: IN0_7 -> IN1_RHDP
- J3 pad 3: IN1_8 -> IN1_2
- J3 pad 4: IN0_8 -> IN1_9
- J3 pad 5: IN1_9 -> IN1_6
- J3 pad 6: IN0_9 -> IN1_0
- J3 pad 7: IN1_2 -> IN1_5
- J3 pad 8: IN0_2 -> IN1_1
- J3 pad 9: IN1_6 -> IN1_4
- U3 pad 1: Net-(J2-Pin_24) -> HVOUT11
- U3 pad 10: Net-(J2-Pin_15) -> HVOUT20
- U3 pad 11: Net-(J2-Pin_14) -> HVOUT21
- U3 pad 12: Net-(J2-Pin_13) -> HVOUT22
- U3 pad 13: Net-(J2-Pin_12) -> HVOUT23
- U3 pad 14: Net-(J2-Pin_11) -> HVOUT24
- U3 pad 16: Net-(J2-Pin_9) -> HVOUT26
- U3 pad 17: Net-(J2-Pin_8) -> HVOUT27
- U3 pad 18: Net-(J2-Pin_7) -> HVOUT28
- U3 pad 19: Net-(J2-Pin_6) -> HVOUT29
- U3 pad 2: Net-(J2-Pin_23) -> HVOUT12
- U3 pad 20: Net-(J2-Pin_5) -> HVOUT30
- U3 pad 21: Net-(J2-Pin_4) -> HVOUT31
- U3 pad 22: Net-(J2-Pin_3) -> HVOUT32
- U3 pad 3: Net-(J2-Pin_22) -> HVOUT13
- U3 pad 4: Net-(J2-Pin_21) -> HVOUT14
- U3 pad 5: Net-(J2-Pin_20) -> HVOUT15
- U3 pad 6: Net-(J2-Pin_19) -> HVOUT16
- U3 pad 7: Net-(J2-Pin_18) -> HVOUT17
- U3 pad 8: Net-(J2-Pin_17) -> HVOUT18
- U3 pad 9: Net-(J2-Pin_16) -> HVOUT19
Other:
- outline, holes or cut-outs redrawn

Commit message: Add files via upload
Parts:
- J2, J3: footprint Connector_PinHeader_1.27mm:PinHeader_2x12_P1.27mm_Vertical -> Connector_FFC-FPC:TE_2-1734839-4_1x24-1MP_P0.5mm_Horizontal
- moved J3 7.45 mm to (142.8, 91.2), turned to 180 degrees
- moved J2 6.87 mm to (142.8, 78.8), turned to 0 degrees
- moved N2 0.59 mm to (149.9, 99.6)
- moved R11 0.59 mm to (149.9, 99.6)
- moved N1 0.59 mm to (136.5, 99.6)
- moved R5 0.59 mm to (136.5, 99.6)
Connections:
- J2 pad 10: HVOUT25 -> HVOUT19
- J2 pad 11: HVOUT17 -> HVOUT20
- J2 pad 12: HVOUT26 -> HVOUT21
- J2 pad 13: HVOUT16 -> HVOUT22
- J2 pad 14: HVOUT27 -> HVOUT23
- J2 pad 15: HVOUT15 -> HVOUT24
- J2 pad 16: HVOUT28 -> HVOUT25
- J2 pad 17: HVOUT14 -> HVOUT26
- J2 pad 18: HVOUT29 -> HVOUT27
- J2 pad 19: HVOUT13 -> HVOUT28
- J2 pad 2: HV -> HVOUT11
- J2 pad 20: HVOUT30 -> HVOUT29
- J2 pad 21: HVOUT12 -> HVOUT30
- J2 pad 23: HVOUT11 -> HVOUT32
- J2 pad 24: HVOUT32 -> HV
- J2 pad 3: HVOUT21 -> HVOUT12
- J2 pad 4: HVOUT22 -> HVOUT13
- J2 pad 5: HVOUT20 -> HVOUT14
- J2 pad 6: HVOUT23 -> HVOUT15
- J2 pad 7: HVOUT19 -> HVOUT16
- J2 pad 8: HVOUT24 -> HVOUT17
- J3 pad 1: IN0_LHDP -> HVe
- J3 pad 10: IN1_7 -> IN1_9
- J3 pad 11: IN0_8 -> IN1_8
- J3 pad 12: IN1_3 -> IN1_RHDPe
- J3 pad 13: IN0_9 -> IN0_LHDPe
- J3 pad 15: IN0_0 -> IN0_6
- J3 pad 16: IN0_6 -> IN0_5
- J3 pad 17: IN0_1 -> IN0_4
- J3 pad 18: IN0_5 -> IN0_8
- J3 pad 19: IN0_7 -> IN0_9
- J3 pad 2: IN1_8 -> IN1_2
- J3 pad 20: IN0_4 -> IN0_3
- J3 pad 21: IN0_3 -> IN0_7
- J3 pad 22: IN1_RHDP -> IN0_1
- J3 pad 23: HVe -> IN0_0
- J3 pad 3: IN1_2 -> IN1_6
- J3 pad 4: IN1_9 -> IN1_5
- J3 pad 5: IN1_6 -> IN1_4
- J3 pad 6: IN1_0 -> IN1_3
- J3 pad 7: IN1_5 -> IN1_7
- J3 pad 9: IN1_4 -> IN1_0
Routing:
- net DCDC: track 0.00 -> 114.0 mm, vias 0 -> 3
- net 3.3VA: track 0.00 -> 74.2 mm, vias 0 -> 5
- net EN: track 0.00 -> 70.9 mm, vias 0 -> 2
- net HV: track 0.00 -> 65.3 mm
- net 5VA: track 0.00 -> 60.8 mm, vias 0 -> 3
- net RST: track 0.00 -> 52.3 mm
- net BAT+: track 0.00 -> 47.3 mm, vias 0 -> 2
- net FB: track 0.00 -> 43.7 mm
- net BOOT: track 0.00 -> 39.6 mm
- net DTR: track 0.00 -> 36.6 mm
- net HVe: track 0.00 -> 34.9 mm, vias 0 -> 2
- net RX0: track 0.00 -> 30.3 mm, vias 0 -> 1
- net WIFI_LED: track 0.00 -> 29.9 mm, vias 0 -> 2
- net Net-(Q2-S): track 0.00 -> 27.8 mm, vias 0 -> 1
- net IN0_5: track 0.00 -> 27.1 mm
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Other:
- outline, holes or cut-outs redrawn

Commit message: Add files via upload
Parts:
- added C2: 100uF, Capacitor_Tantalum_SMD:CP_EIA-1608-08_AVX-J, F.Cu at (129.8, 66.9)
- added D2: 1N4148W, Diode_SMD:D_SOD-123, F.Cu at (129.4, 70.0)
- added D3: 1N4148W, Diode_SMD:D_SOD-123, F.Cu at (127.7, 71.8)
- R15, U5: moved to B.Cu
- moved R15 16.4 mm to (131.0, 74.1), turned to 135 degrees
- moved C1 10.6 mm to (130.1, 56.4), turned to -45 degrees
- moved C10 10.2 mm to (137.1, 63.4), turned to -45 degrees
- moved C9 9.37 mm to (128.5, 71.5), turned to -45 degrees
- moved U5 8.99 mm to (132.3, 67.9), turned to 45 degrees
- moved C11 7.98 mm to (137.5, 51.5)
- moved C12 7.98 mm to (135.4, 53.7)
- moved R17 5.82 mm to (145.0, 56.4), turned to -45 degrees
- moved R16 4.00 mm to (146.4, 55.0)
- moved C8 3.11 mm to (151.7, 51.6)
- moved J2 2.55 mm to (142.8, 88.6)
- moved N1 2.55 mm to (136.5, 97.1)
- moved N2 2.55 mm to (149.9, 97.1)
- moved R11 2.55 mm to (149.9, 97.1)
- moved R5 2.55 mm to (136.5, 97.1)
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- renumbered C9 to C10, C10 to C11, C11 to C12, C12 to C13, C2 to C3, C3 to C4, C4 to C5, C5 to C6, C6 to C7, C7 to C8, C8 to C9, D2 to D4, D3 to D5, D4 to D6, D5 to D7, D6 to D8, J3 to J2, J2 to J3
Connections:
- J1 pad 1: VIN -> Net-(D2-A)
- Q3 pad 2: IO0 -> BOOT
Routing:
- net BAT-: track 0.00 -> 217.7 mm, vias 2 -> 6
- net EN: track 70.9 -> 49.9 mm, vias 2 -> 6
- net Net-(D2-A): track 0.00 -> 16.6 mm
- net WIFI_LED: track 29.9 -> 45.4 mm, vias 2 -> 4
- net DCDC: track 114.0 -> 128.7 mm, vias 3 -> 5
- net FB: track 43.7 -> 32.5 mm
- net Net-(Q4-B): track 10.1 -> 19.7 mm, vias 1 -> 3
- net RX0: track 30.3 -> 39.3 mm, vias 1 -> 4
- net SW2: track 25.1 -> 33.8 mm, vias 2 -> 1
- net TX0: track 24.6 -> 33.0 mm, vias 1 -> 2
- net BAT+: track 47.3 -> 39.0 mm
- net BOOT: track 39.6 -> 32.0 mm, vias 0 -> 2
- net STAT: track 19.7 -> 12.7 mm, vias 1 -> 0
- net Net-(Q5-B): track 12.7 -> 5.80 mm
- net RST: track 52.3 -> 58.8 mm, vias 0 -> 4
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Other:
- board size 49.8 x 67.6 mm -> 49.7 x 64.8 mm

Commit message: Add files via upload
Parts:
- moved R5 10.1 mm to (132.8, 87.8), turned to -135 degrees
- moved R11 10.0 mm to (153.5, 87.8), turned to -45 degrees
- moved N1 2.62 mm to (136.5, 94.5)
- moved N2 2.62 mm to (149.9, 94.5)
- moved J2 1.00 mm to (142.8, 87.6)
Routing:
- net IN1_0: track 10.1 -> 29.5 mm, vias 1 -> 2
- net IN0_0: track 4.53 -> 18.0 mm, vias 1 -> 0
- net IN0_5: track 27.7 -> 14.8 mm
- net IN0_7: track 16.1 -> 7.19 mm
- net IN1_5: track 14.3 -> 22.9 mm
- net IN0_3: track 10.2 -> 17.4 mm, vias 0 -> 1
- net IN1_4: track 15.2 -> 9.12 mm, vias 1 -> 0
- net FB: track 32.5 -> 38.1 mm
- net IN1_3: track 11.6 -> 16.9 mm, vias 1 -> 2
- net IN1_6: track 25.7 -> 23.0 mm, vias 0 -> 2
- net Net-(N1-PadA): track 2.93 -> 5.31 mm
- net DTR: track 40.7 -> 38.3 mm
- net IN0_4: track 16.2 -> 14.0 mm
- net IN1_2: track 15.2 -> 13.2 mm, vias 0 -> 2
- net STAT: track 12.7 -> 10.9 mm
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Other:
- board size 49.7 x 64.8 mm -> 49.7 x 63.1 mm
